File: NBPD EAGLE/Layout.sch (EAGLE design)
At the start: 8 parts, among them IC1 4040N, IC2 4040N, IC3 4017N, IC4 4017N, IC5 4017N, IC6 4017N, U1 LM317K, Y1 ACHL-32.768MHZ-EK

Commit message: Add files via upload
Parts:
- added IC7: 7818TV, linear:7818TV
Connections:
- net 5V: now also IC7.VO
- net N$1: now also IC7.GND
Changed lines of the file:
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@@
 <layer number="97" name="Info" color="7" fill="1" visible="yes" active="yes"/>
 <layer number="98" name="Guide" color="6" fill="1" visible="yes" active="yes"/>
+<layer number="99" name="SpiceOrder" color="7" fill="1" visible="yes" active="yes"/>
 </layers>
 <schematic xreflabel="%F%N/%S.%C%R" xrefpart="/%S.%C%R">
@@
 <part name="Y1" library="ACHL-32.768MHZ-EK" deviceset="ACHL-32.768MHZ-EK" device=""/>
 <part name="U1" library="LM317K" deviceset="LM317K" device=""/>
+<part name="R1" library="docu-dummy" library_urn="urn:adsk.eagle:library:215" deviceset="R" device=""/>
+<part name="R2" library="docu-dummy" library_urn="urn:adsk.eagle:library:215" deviceset="R" device=""/>
+<part name="R3" library="docu-dummy" library_urn="urn:adsk.eagle:library:215" deviceset="R" device=""/>
+<part name="X_1" library="ngspice-simulation" library_urn="urn:adsk.eagle:library:527439" deviceset="GND" device=""/>
+<part name="IC7" library="linear" library_urn="urn:adsk.eagle:library:262" deviceset="78*" device="TV" package3d_urn="urn:adsk.eagle:package:16417/1" technology="18"/>
 </parts>
 <sheets>
@@
 <attribute name="VALUE" x="55.74618125" y="91.5726" size="2.08553125" layer="96" ratio="10" rot="SR0"/>
 </instance>
+<instance part="R1" gate="G$1" x="121.92" y="-38.1" smashed="yes" rot="R90"/>
+<instance part="R2" gate="G$1" x="78.74" y="-38.1" smashed="yes" rot="R90"/>
+<instance part="R3" gate="G$1" x="35.56" y="-38.1" smashed="yes" rot="R270"/>
+<instance part="X_1" gate="G$1" x="10.16" y="-58.42" smashed="yes"/>
+<instance part="IC7" gate="A1" x="127" y="99.06" smashed="yes">
+<attribute name="NAME" x="119.38" y="104.775" size="1.778" layer="95"/>
+<attribute name="VALUE" x="119.38" y="102.235" size="1.778" layer="96"/>
+</instance>
 </instances>
 <busses>
@@
 <pinref part="Y1" gate="G$1" pin="GND"/>
 <wire x1="-111.76" y1="86.36" x2="-142.24" y2="86.36" width="0.1524" layer="91"/>
-<wire x1="-142.24" y1="86.36" x2="-142.24" y2="12.7" width="0.1524" layer="91"/>
+<wire x1="-142.24" y1="86.36" x2="-142.24" y2="15.24" width="0.1524" layer="91"/>
+<wire x1="-142.24" y1="15.24" x2="-142.24" y2="12.7" width="0.1524" layer="91"/>
+<wire x1="-142.24" y1="15.24" x2="-152.4" y2="15.24" width="0.1524" layer="91"/>
+<junction x="-142.24" y="15.24"/>
+<pinref part="X_1" gate="G$1" pin="0"/>
+<wire x1="10.16" y1="-58.42" x2="10.16" y2="-53.34" width="0.1524" layer="91"/>
+<wire x1="10.16" y1="-53.34" x2="10.16" y2="-43.18" width="0.1524" layer="91"/>
+<pinref part="IC7" gate="A1" pin="GND"/>
+<wire x1="127" y1="91.44" x2="127" y2="-27.94" width="0.1524" layer="91"/>
+<wire x1="127" y1="-27.94" x2="152.4" y2="-27.94" width="0.1524" layer="91"/>
+<wire x1="152.4" y1="-27.94" x2="152.4" y2="-53.34" width="0.1524" layer="91"/>
+<wire x1="152.4" y1="-53.34" x2="10.16" y2="-53.34" width="0.1524" layer="91"/>
+<junction x="10.16" y="-53.34"/>
+<wire x1="10.16" y1="-43.18" x2="121.92" y2="-43.18" width="0.1524" layer="91"/>
+<wire x1="-152.4" y1="15.24" x2="-152.4" y2="-53.34" width="0.1524" layer="91"/>
+<wire x1="-152.4" y1="-53.34" x2="10.16" y2="-53.34" width="0.1524" layer="91"/>
 </segment>
 </net>
@@
 <wire x1="-78.74" y1="48.26" x2="-78.74" y2="0" width="0.1524" layer="91"/>
 </segment>
+<segment>
+<pinref part="IC7" gate="A1" pin="VO"/>
+<wire x1="137.16" y1="99.06" x2="137.16" y2="0" width="0.1524" layer="91"/>
+<wire x1="137.16" y1="0" x2="116.84" y2="0" width="0.1524" layer="91"/>
+</segment>
 </net>
 <net name="6V" class="0">
@@
 <pinref part="IC6" gate="P" pin="VDD"/>
 <wire x1="10.16" y1="63.5" x2="0" y2="63.5" width="0.1524" layer="91"/>
-<wire x1="0" y1="63.5" x2="0" y2="-15.24" width="0.1524" layer="91"/>
-</segment>
-<segment>
+</segment>
+<segment>

Commit message: Fix connection
Connections:
- new net N$8: IC7.VI
Other:
- note added: "9V IN"
Changed lines of the file:
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@@
 <sheet>
 <plain>
+<text x="104.14" y="101.6" size="1.778" layer="91">9V IN</text>
 </plain>
 <instances>
@@
 </segment>
 <segment>
-<pinref part="IC6" gate="P" pin="VDD"/>
-<wire x1="10.16" y1="63.5" x2="0" y2="63.5" width="0.1524" layer="91"/>
-</segment>
-<segment>
 <pinref part="IC4" gate="P" pin="VDD"/>
 <wire x1="50.8" y1="63.5" x2="38.1" y2="63.5" width="0.1524" layer="91"/>
@@
 <wire x1="144.78" y1="116.84" x2="144.78" y2="-15.24" width="0.1524" layer="91"/>
 <wire x1="144.78" y1="-15.24" x2="114.3" y2="-15.24" width="0.1524" layer="91"/>
+</segment>
+<segment>
+<pinref part="IC6" gate="P" pin="VDD"/>
+<wire x1="10.16" y1="63.5" x2="0" y2="63.5" width="0.1524" layer="91"/>
+<wire x1="0" y1="63.5" x2="0" y2="-15.24" width="0.1524" layer="91"/>
 </segment>
 </net>
@@
 </segment>
 </net>
+<net name="N$8" class="0">
+<segment>
+<pinref part="IC7" gate="A1" pin="VI"/>
+<wire x1="116.84" y1="99.06" x2="106.68" y2="99.06" width="0.1524" layer="91"/>
+</segment>
+</net>

Commit message: Add files via upload
Connections:
- new net N$9: U1.ADJ
- net 5V: now also IC3P.VDD, IC4P.VDD, IC5P.VDD, IC6P.VDD; no longer IC1P.VDD, IC2P.VDD
- net 6V: now also IC1P.VDD, IC2P.VDD; no longer IC3P.VDD, IC4P.VDD, IC5P.VDD, IC6P.VDD
- net N$1: now also IC4A.RES

Commit message: Update resistor
Connections:
- new net N$10: IC6P.VDD
- new net N$11: IC4P.VDD
- new net N$12: IC5P.VDD
- new net N$13: IC3P.VDD
- net 5V: no longer IC3P.VDD, IC4P.VDD, IC5P.VDD, IC6P.VDD
Other:
- note added: "220Ω"
- note added: "330Ω"
- note added: "GND"
Changed lines of the file:
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@@
 <part name="X_1" library="ngspice-simulation" library_urn="urn:adsk.eagle:library:527439" deviceset="GND" device=""/>
 <part name="IC7" library="linear" library_urn="urn:adsk.eagle:library:262" deviceset="78*" device="TV" package3d_urn="urn:adsk.eagle:package:16417/1" technology="18"/>
-<part name="R4" library="docu-dummy" library_urn="urn:adsk.eagle:library:215" deviceset="R" device=""/>
+<part name="R4" library="docu-dummy" library_urn="urn:adsk.eagle:library:215" deviceset="R" device="" value="220"/>
 <part name="R5" library="docu-dummy" library_urn="urn:adsk.eagle:library:215" deviceset="R" device=""/>
 <part name="C1" library="docu-dummy" library_urn="urn:adsk.eagle:library:215" deviceset="C" device=""/>
@@
 <part name="C5" library="docu-dummy" library_urn="urn:adsk.eagle:library:215" deviceset="C" device=""/>
 <part name="C6" library="docu-dummy" library_urn="urn:adsk.eagle:library:215" deviceset="C" device=""/>
+<part name="C7" library="docu-dummy" library_urn="urn:adsk.eagle:library:215" deviceset="C" device=""/>
+<part name="C8" library="docu-dummy" library_urn="urn:adsk.eagle:library:215" deviceset="C" device=""/>
+<part name="C9" library="docu-dummy" library_urn="urn:adsk.eagle:library:215" deviceset="C" device=""/>
+<part name="C10" library="docu-dummy" library_urn="urn:adsk.eagle:library:215" deviceset="C" device=""/>
 </parts>
 <sheets>
@@
 <plain>
 <text x="104.14" y="101.6" size="1.778" layer="91">9V IN</text>
+<text x="-152.4" y="17.78" size="1.778" layer="91">GND</text>
+<text x="35.56" y="88.9" size="1.778" layer="91">220Ω</text>
+<text x="33.02" y="96.52" size="1.778" layer="91">330Ω</text>
 </plain>
 <instances>
@@
 <instance part="C5" gate="G$1" x="-134.62" y="38.1" smashed="yes"/>
 <instance part="C6" gate="G$1" x="-83.82" y="22.86" smashed="yes"/>
+<instance part="C7" gate="G$1" x="0" y="53.34" smashed="yes"/>
+<instance part="C8" gate="G$1" x="38.1" y="55.88" smashed="yes"/>
+<instance part="C9" gate="G$1" x="81.28" y="53.34" smashed="yes"/>
+<instance part="C10" gate="G$1" x="-40.64" y="53.34" smashed="yes"/>
 </instances>
 <busses>
@@
 </segment>
 <segment>
-<pinref part="IC3" gate="P" pin="VDD"/>
-<wire x1="-30.48" y1="60.96" x2="-40.64" y2="60.96" width="0.1524" layer="91"/>
-<wire x1="-40.64" y1="60.96" x2="-40.64" y2="0" width="0.1524" layer="91"/>
-<junction x="-40.64" y="0"/>
-</segment>
-<segment>
-<pinref part="IC6" gate="P" pin="VDD"/>
-<wire x1="10.16" y1="63.5" x2="0" y2="63.5" width="0.1524" layer="91"/>
-<wire x1="0" y1="63.5" x2="0" y2="0" width="0.1524" layer="91"/>
-<junction x="0" y="0"/>
-</segment>
-<segment>
-<pinref part="IC4" gate="P" pin="VDD"/>
-<wire x1="50.8" y1="63.5" x2="38.1" y2="63.5" width="0.1524" layer="91"/>
-<wire x1="38.1" y1="63.5" x2="38.1" y2="0" width="0.1524" layer="91"/>
-<junction x="38.1" y="0"/>
-</segment>
-<segment>
-<pinref part="IC5" gate="P" pin="VDD"/>
-<wire x1="96.52" y1="60.96" x2="81.28" y2="60.96" width="0.1524" layer="91"/>
-<wire x1="81.28" y1="60.96" x2="81.28" y2="0" width="0.1524" layer="91"/>
-<junction x="81.28" y="0"/>
+<wire x1="0" y1="48.26" x2="0" y2="0" width="0.1524" layer="91"/>
+</segment>
+<segment>
+<wire x1="38.1" y1="50.8" x2="38.1" y2="0" width="0.1524" layer="91"/>
+</segment>
+<segment>
+<wire x1="81.28" y1="48.26" x2="81.28" y2="0" width="0.1524" layer="91"/>
+</segment>
+<segment>
+<wire x1="-40.64" y1="48.26" x2="-40.64" y2="0" width="0.1524" layer="91"/>
 </segment>
 </net>
@@
 </segment>
 </net>
+<net name="N$10" class="0">
+<segment>
+<pinref part="IC6" gate="P" pin="VDD"/>
+<wire x1="10.16" y1="63.5" x2="0" y2="63.5" width="0.1524" layer="91"/>
+<wire x1="0" y1="63.5" x2="0" y2="55.88" width="0.1524" layer="91"/>
+</segment>
+</net>
+<net name="N$11" class="0">
+<segment>
+<pinref part="IC4" gate="P" pin="VDD"/>
+<wire x1="50.8" y1="63.5" x2="38.1" y2="63.5" width="0.1524" layer="91"/>
+<wire x1="38.1" y1="63.5" x2="38.1" y2="55.88" width="0.1524" layer="91"/>
+</segment>
+</net>
+<net name="N$12" class="0">
+<segment>
+<pinref part="IC5" gate="P" pin="VDD"/>
+<wire x1="96.52" y1="60.96" x2="81.28" y2="60.96" width="0.1524" layer="91"/>
+<wire x1="81.28" y1="60.96" x2="81.28" y2="55.88" width="0.1524" layer="91"/>
+</segment>
+</net>
+<net name="N$13" class="0">
+<segment>
+<pinref part="IC3" gate="P" pin="VDD"/>
+<wire x1="-30.48" y1="60.96" x2="-40.64" y2="60.96" width="0.1524" layer="91"/>
+<wire x1="-40.64" y1="60.96" x2="-40.64" y2="55.88" width="0.1524" layer="91"/>
+</segment>
+</net>

Commit message: Add text labels
Other:
- note added: ".1 µF capacitors attached to all IC power"
- note added: ".33 µF"
- note added: "1 µF"
- note added: "1K Ω"
Changed lines of the file:
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@@
 <text x="35.56" y="88.9" size="1.778" layer="91">220Ω</text>
 <text x="33.02" y="96.52" size="1.778" layer="91">330Ω</text>
+<text x="-22.86" y="73.66" size="1.778" layer="91">1K Ω</text>
+<text x="0" y="73.66" size="1.778" layer="91">1K Ω</text>
+<text x="101.6" y="93.98" size="1.778" layer="91">.33 µF</text>
+<text x="129.54" y="78.74" size="1.778" layer="91">1 µF</text>
+<text x="-91.44" y="119.38" size="1.778" layer="91">.1 µF capacitors attached to all IC power</text>
 </plain>
 <instances>

Commit message: Update Schematic
Other:
- note added: ".1 µF capacitors attached to all IC power input"
- note removed: ".1 µF capacitors attached to all IC power"
Changed lines of the file:
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@@
 <text x="101.6" y="93.98" size="1.778" layer="91">.33 µF</text>
 <text x="129.54" y="78.74" size="1.778" layer="91">1 µF</text>
-<text x="-91.44" y="119.38" size="1.778" layer="91">.1 µF capacitors attached to all IC power</text>
+<text x="-91.44" y="119.38" size="1.778" layer="91">.1 µF capacitors attached to all IC power input</text>
 </plain>
 <instances>

Commit message: Add files via upload
Connections:
- removed net N$10: IC6P.VDD
- removed net N$11: IC4P.VDD
- removed net N$12: IC5P.VDD
- removed net N$13: IC3P.VDD
- net 5V: now also IC3P.VDD, IC4P.VDD, IC5P.VDD, IC6P.VDD
- net N$1: now also IC1P.VSS, IC2P.VSS, IC3P.VSS, IC4P.VSS, IC5P.VSS, IC6P.VSS
Changed lines of the file:
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@@
 <instance part="C5" gate="G$1" x="-134.62" y="38.1" smashed="yes"/>
 <instance part="C6" gate="G$1" x="-83.82" y="22.86" smashed="yes"/>
-<instance part="C7" gate="G$1" x="0" y="53.34" smashed="yes"/>
+<instance part="C7" gate="G$1" x="-2.54" y="53.34" smashed="yes"/>
 <instance part="C8" gate="G$1" x="38.1" y="55.88" smashed="yes"/>
 <instance part="C9" gate="G$1" x="81.28" y="53.34" smashed="yes"/>
-<instance part="C10" gate="G$1" x="-40.64" y="53.34" smashed="yes"/>
+<instance part="C10" gate="G$1" x="-43.18" y="53.34" smashed="yes"/>
 </instances>
 <busses>
@@
 <wire x1="-30.48" y1="33.02" x2="-38.1" y2="33.02" width="0.1524" layer="91"/>
 <wire x1="-38.1" y1="33.02" x2="-38.1" y2="12.7" width="0.1524" layer="91"/>
+<junction x="-38.1" y="12.7"/>
 </segment>
 <segment>
@@
 <junction x="50.8" y="12.7"/>
 </segment>
+<segment>
+<pinref part="IC1" gate="P" pin="VSS"/>
+<wire x1="-111.76" y1="35.56" x2="-121.92" y2="35.56" width="0.1524" layer="91"/>
+<wire x1="-121.92" y1="35.56" x2="-121.92" y2="12.7" width="0.1524" layer="91"/>
+<junction x="-121.92" y="12.7"/>
+</segment>
+<segment>
+<pinref part="IC2" gate="P" pin="VSS"/>
+<wire x1="-68.58" y1="33.02" x2="-73.66" y2="33.02" width="0.1524" layer="91"/>
+<wire x1="-73.66" y1="33.02" x2="-73.66" y2="12.7" width="0.1524" layer="91"/>
+<junction x="-73.66" y="12.7"/>
+</segment>
+<segment>
+<pinref part="IC3" gate="P" pin="VSS"/>
+<wire x1="-30.48" y1="45.72" x2="-35.56" y2="45.72" width="0.1524" layer="91"/>
+<wire x1="-35.56" y1="45.72" x2="-35.56" y2="12.7" width="0.1524" layer="91"/>
+<junction x="-35.56" y="12.7"/>
+</segment>
+<segment>
+<pinref part="IC6" gate="P" pin="VSS"/>
+<wire x1="10.16" y1="48.26" x2="5.08" y2="48.26" width="0.1524" layer="91"/>
+<wire x1="5.08" y1="48.26" x2="5.08" y2="12.7" width="0.1524" layer="91"/>
+<junction x="5.08" y="12.7"/>
+</segment>
+<segment>
+<pinref part="IC4" gate="P" pin="VSS"/>
+<wire x1="50.8" y1="48.26" x2="45.72" y2="48.26" width="0.1524" layer="91"/>
+<wire x1="45.72" y1="48.26" x2="45.72" y2="12.7" width="0.1524" layer="91"/>
+<junction x="45.72" y="12.7"/>
+</segment>
+<segment>
+<pinref part="IC5" gate="P" pin="VSS"/>
+<wire x1="96.52" y1="45.72" x2="88.9" y2="45.72" width="0.1524" layer="91"/>
+<wire x1="88.9" y1="45.72" x2="88.9" y2="12.7" width="0.1524" layer="91"/>
+<junction x="88.9" y="12.7"/>
+</segment>
+<segment>
+<wire x1="-43.18" y1="48.26" x2="-43.18" y2="12.7" width="0.1524" layer="91"/>
+<junction x="-43.18" y="12.7"/>
+</segment>
+<segment>
+<wire x1="-2.54" y1="48.26" x2="-2.54" y2="12.7" width="0.1524" layer="91"/>
+<junction x="-2.54" y="12.7"/>
+</segment>
+<segment>
+<wire x1="38.1" y1="50.8" x2="38.1" y2="12.7" width="0.1524" layer="91"/>
+<junction x="38.1" y="12.7"/>
+</segment>
+<segment>
+<wire x1="81.28" y1="48.26" x2="81.28" y2="12.7" width="0.1524" layer="91"/>
+<junction x="81.28" y="12.7"/>
+</segment>
 </net>
 <net name="N$2" class="0">
@@
 </segment>
 <segment>
-<wire x1="0" y1="48.26" x2="0" y2="0" width="0.1524" layer="91"/>
-</segment>
-<segment>
-<wire x1="38.1" y1="50.8" x2="38.1" y2="0" width="0.1524" layer="91"/>
-</segment>
-<segment>
-<wire x1="81.28" y1="48.26" x2="81.28" y2="0" width="0.1524" layer="91"/>
-</segment>
-<segment>
-<wire x1="-40.64" y1="48.26" x2="-40.64" y2="0" width="0.1524" layer="91"/>
+<pinref part="IC3" gate="P" pin="VDD"/>
+<wire x1="-30.48" y1="60.96" x2="-40.64" y2="60.96" width="0.1524" layer="91"/>
+<wire x1="-40.64" y1="60.96" x2="-40.64" y2="55.88" width="0.1524" layer="91"/>
+<junction x="-40.64" y="0"/>
+<wire x1="-40.64" y1="55.88" x2="-40.64" y2="0" width="0.1524" layer="91"/>
+<wire x1="-43.18" y1="55.88" x2="-40.64" y2="55.88" width="0.1524" layer="91"/>
+<junction x="-40.64" y="55.88"/>
+</segment>
+<segment>
+<pinref part="IC6" gate="P" pin="VDD"/>
+<wire x1="10.16" y1="63.5" x2="0" y2="63.5" width="0.1524" layer="91"/>
+<wire x1="0" y1="63.5" x2="0" y2="55.88" width="0.1524" layer="91"/>
+<junction x="0" y="0"/>
+<wire x1="0" y1="55.88" x2="0" y2="0" width="0.1524" layer="91"/>
+<wire x1="-2.54" y1="55.88" x2="0" y2="55.88" width="0.1524" layer="91"/>
+<junction x="0" y="55.88"/>
+</segment>
+<segment>
+<pinref part="IC4" gate="P" pin="VDD"/>
+<wire x1="50.8" y1="63.5" x2="43.18" y2="63.5" width="0.1524" layer="91"/>
+<wire x1="43.18" y1="63.5" x2="43.18" y2="60.96" width="0.1524" layer="91"/>
+<junction x="43.18" y="0"/>
+<wire x1="43.18" y1="60.96" x2="43.18" y2="0" width="0.1524" layer="91"/>
+<wire x1="38.1" y1="58.42" x2="38.1" y2="60.96" width="0.1524" layer="91"/>
+<wire x1="38.1" y1="60.96" x2="43.18" y2="60.96" width="0.1524" layer="91"/>
+<junction x="43.18" y="60.96"/>
+</segment>
+<segment>
+<pinref part="IC5" gate="P" pin="VDD"/>
+<wire x1="96.52" y1="60.96" x2="86.36" y2="60.96" width="0.1524" layer="91"/>
+<wire x1="86.36" y1="60.96" x2="86.36" y2="55.88" width="0.1524" layer="91"/>
+<junction x="86.36" y="0"/>
+<wire x1="86.36" y1="55.88" x2="86.36" y2="0" width="0.1524" layer="91"/>
+<wire x1="81.28" y1="55.88" x2="86.36" y2="55.88" width="0.1524" layer="91"/>
+<junction x="86.36" y="55.88"/>
 </segment>
 </net>
@@
 </segment>
 </net>
-<net name="N$10" class="0">
-<segment>
-<pinref part="IC6" gate="P" pin="VDD"/>
-<wire x1="10.16" y1="63.5" x2="0" y2="63.5" width="0.1524" layer="91"/>
-<wire x1="0" y1="63.5" x2="0" y2="55.88" width="0.1524" layer="91"/>
-</segment>
-</net>
-<net name="N$11" class="0">
-<segment>
-<pinref part="IC4" gate="P" pin="VDD"/>
-<wire x1="50.8" y1="63.5" x2="38.1" y2="63.5" width="0.1524" layer="91"/>
-<wire x1="38.1" y1="63.5" x2="38.1" y2="55.88" width="0.1524" layer="91"/>
-</segment>
-</net>
-<net name="N$12" class="0">
-<segment>
-<pinref part="IC5" gate="P" pin="VDD"/>
-<wire x1="96.52" y1="60.96" x2="81.28" y2="60.96" width="0.1524" layer="91"/>
-<wire x1="81.28" y1="60.96" x2="81.28" y2="55.88" width="0.1524" layer="91"/>
-</segment>
-</net>
-<net name="N$13" class="0">
-<segment>
-<pinref part="IC3" gate="P" pin="VDD"/>
-<wire x1="-30.48" y1="60.96" x2="-40.64" y2="60.96" width="0.1524" layer="91"/>
-<wire x1="-40.64" y1="60.96" x2="-40.64" y2="55.88" width="0.1524" layer="91"/>
-</segment>
-</net>

Commit message: Move Locations
Other:
- note added: "CATHODES OF LEDs"
- note added: "OUTPUTS OF 4017 CONNECTED TO ANODE OF LEDs"
Changed lines of the file:
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@@
 <text x="129.54" y="78.74" size="1.778" layer="91">1 µF</text>
 <text x="-91.44" y="119.38" size="1.778" layer="91">.1 µF capacitors attached to all IC power input</text>
+<text x="25.4" y="-30.48" size="1.778" layer="91">CATHODES OF LEDs</text>
+<text x="66.04" y="-30.48" size="1.778" layer="91">CATHODES OF LEDs</text>
+<text x="111.76" y="-30.48" size="1.778" layer="91">CATHODES OF LEDs</text>
+<text x="-88.9" y="109.22" size="1.778" layer="91">OUTPUTS OF 4017
+CONNECTED TO ANODE OF LEDs</text>
 </plain>
 <instances>
@@
 </drawing>
 <compatibility>
+<note version="6.3" minversion="6.2.2" severity="warning">
+Since Version 6.2.2 text objects can contain more than one line,
+which will not be processed correctly with this version.
+</note>
 <note version="8.2" severity="warning">
 Since Version 8.2, EAGLE supports online libraries. The ids
