File: NBPD EAGLE/Layout.sch (EAGLE design)
At the start: 28 parts, among them IC1 4040N, IC2 4040N, IC3 4017N, IC4 4017N, IC5 4017N, IC6 4017N, IC7 7818TV, U1 LM317K, Y1 ACHL-32.768MHZ-EK

Commit message: 10 HZ 1 HZ
Parts:
- added LED20: SSL-LX5093TC, SSL-LX5093TC:SSL-LX5093TC
Connections:
- new net 10HZGROUND: LED11.K, LED12.K, LED13.K, LED14.K, LED15.K, LED16.K, LED17.K, LED18.K, LED19.K, LED20.K
- new net N$20: IC4A.Q0, LED11.A
- new net N$21: IC4A.Q1, LED12.A
- new net N$22: IC4A.Q2, LED13.A
- new net N$23: IC4A.Q3, LED14.A
- new net N$24: IC4A.Q4, LED15.A
- new net N$25: IC4A.Q5, LED16.A
- new net N$26: IC4A.Q6, LED17.A
- new net N$27: IC4A.Q7, LED18.A
- new net N$28: IC4A.Q8, LED19.A
- new net N$29: IC4A.Q9, LED20.A
- net N$3: now also IC3A.CO; no longer IC3A.Q9
- net N$4: now also IC6A.CO; no longer IC6A.Q9
- net N$5: now also IC4A.CO; no longer IC4A.Q9
Other:
- moved on the sheet: IC4, IC4P

Commit message: Third LED
Parts:
- added LED21, LED22, LED23, LED24, LED25, LED26, LED27, LED28, LED29, LED30: SSL-LX5093TC, SSL-LX5093TC:SSL-LX5093TC
- added R1, R2, R3: 220, rcl:R-US_0207/12
- added R4: 220, rcl:R-US_0309/12
- added R5, R6, R7: (no value), rcl:R-US_0309/12
Connections:
- net 10HZGROUND: now also LED21.K, LED22.K, LED23.K, LED24.K, LED25.K, LED26.K, LED27.K, LED28.K, LED29.K, LED30.K
- net N$1: now also R3.2
Changed lines of the file:
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@@
 <?xml version="1.0" encoding="utf-8"?>
 <!DOCTYPE eagle SYSTEM "eagle.dtd">
-<eagle version="9.3.0">
+<eagle version="8.4.3">
 <drawing>
 <settings>
@@
 <part name="Y1" library="ACHL-32.768MHZ-EK" deviceset="ACHL-32.768MHZ-EK" device=""/>
 <part name="U1" library="LM317K" deviceset="LM317K" device=""/>
-<part name="R1" library="docu-dummy" library_urn="urn:adsk.eagle:library:215" deviceset="R" device=""/>
-<part name="R2" library="docu-dummy" library_urn="urn:adsk.eagle:library:215" deviceset="R" device=""/>
-<part name="R3" library="docu-dummy" library_urn="urn:adsk.eagle:library:215" deviceset="R" device=""/>
+<part name="R1" library="rcl" library_urn="urn:adsk.eagle:library:334" deviceset="R-US_" device="0207/12" package3d_urn="urn:adsk.eagle:package:23489/1" value="220">
+<attribute name="R6" value="220"/>
+</part>
+<part name="R2" library="rcl" library_urn="urn:adsk.eagle:library:334" deviceset="R-US_" device="0207/12" package3d_urn="urn:adsk.eagle:package:23489/1" value="220">
+<attribute name="R5" value="220"/>
+</part>
 <part name="X_1" library="ngspice-simulation" library_urn="urn:adsk.eagle:library:527439" deviceset="GND" device=""/>
 <part name="IC7" library="linear" library_urn="urn:adsk.eagle:library:262" deviceset="78*" device="TV" package3d_urn="urn:adsk.eagle:package:16417/1" technology="18"/>
-<part name="R4" library="docu-dummy" library_urn="urn:adsk.eagle:library:215" deviceset="R" device="" value="220"/>
-<part name="R5" library="docu-dummy" library_urn="urn:adsk.eagle:library:215" deviceset="R" device=""/>
+<part name="R4" library="rcl" library_urn="urn:adsk.eagle:library:334" deviceset="R-US_" device="0309/12" package3d_urn="urn:adsk.eagle:package:23571/1" value="220"/>
+<part name="R5" library="rcl" library_urn="urn:adsk.eagle:library:334" deviceset="R-US_" device="0309/12" package3d_urn="urn:adsk.eagle:package:23571/1"/>
 <part name="C1" library="docu-dummy" library_urn="urn:adsk.eagle:library:215" deviceset="C" device=""/>
 <part name="C2" library="docu-dummy" library_urn="urn:adsk.eagle:library:215" deviceset="C" device=""/>
-<part name="R6" library="docu-dummy" library_urn="urn:adsk.eagle:library:215" deviceset="R" device=""/>
-<part name="R7" library="docu-dummy" library_urn="urn:adsk.eagle:library:215" deviceset="R" device=""/>
+<part name="R6" library="rcl" library_urn="urn:adsk.eagle:library:334" deviceset="R-US_" device="0309/12" package3d_urn="urn:adsk.eagle:package:23571/1"/>
+<part name="R7" library="rcl" library_urn="urn:adsk.eagle:library:334" deviceset="R-US_" device="0309/12" package3d_urn="urn:adsk.eagle:package:23571/1"/>
 <part name="C3" library="docu-dummy" library_urn="urn:adsk.eagle:library:215" deviceset="C" device=""/>
 <part name="C4" library="docu-dummy" library_urn="urn:adsk.eagle:library:215" deviceset="C" device=""/>
@@
 <part name="LED19" library="SSL-LX5093TC" deviceset="SSL-LX5093TC" device=""/>
 <part name="LED20" library="SSL-LX5093TC" deviceset="SSL-LX5093TC" device=""/>
+<part name="R3" library="rcl" library_urn="urn:adsk.eagle:library:334" deviceset="R-US_" device="0207/12" package3d_urn="urn:adsk.eagle:package:23489/1" value="220">
+<attribute name="R4" value="220"/>
+</part>
+<part name="LED21" library="SSL-LX5093TC" deviceset="SSL-LX5093TC" device=""/>
+<part name="LED22" library="SSL-LX5093TC" deviceset="SSL-LX5093TC" device=""/>
+<part name="LED23" library="SSL-LX5093TC" deviceset="SSL-LX5093TC" device=""/>
+<part name="LED24" library="SSL-LX5093TC" deviceset="SSL-LX5093TC" device=""/>
+<part name="LED25" library="SSL-LX5093TC" deviceset="SSL-LX5093TC" device=""/>
+<part name="LED26" library="SSL-LX5093TC" deviceset="SSL-LX5093TC" device=""/>
+<part name="LED27" library="SSL-LX5093TC" deviceset="SSL-LX5093TC" device=""/>
+<part name="LED28" library="SSL-LX5093TC" deviceset="SSL-LX5093TC" device=""/>
+<part name="LED29" library="SSL-LX5093TC" deviceset="SSL-LX5093TC" device=""/>
+<part name="LED30" library="SSL-LX5093TC" deviceset="SSL-LX5093TC" device=""/>
 </parts>
 <sheets>
@@
 <attribute name="VALUE" x="55.74618125" y="91.5726" size="2.08553125" layer="96" ratio="10" rot="SR0"/>
 </instance>
-<instance part="R1" gate="G$1" x="121.92" y="-63.5" smashed="yes" rot="R90"/>
-<instance part="R2" gate="G$1" x="66.04" y="-63.5" smashed="yes" rot="R90"/>
-<instance part="R3" gate="G$1" x="35.56" y="-63.5" smashed="yes" rot="R90"/>
+<instance part="R1" gate="G$1" x="121.92" y="-63.5" smashed="yes" rot="R90">
+<attribute name="R6" x="121.92" y="-63.5" size="1.778" layer="96" rot="R90"/>
+</instance>
+<instance part="R2" gate="G$1" x="66.04" y="-63.5" smashed="yes" rot="R90">
+<attribute name="R5" x="66.04" y="-63.5" size="1.778" layer="96" rot="R90"/>
+</instance>
 <instance part="X_1" gate="G$1" x="10.16" y="-58.42" smashed="yes"/>
 <instance part="IC7" gate="A1" x="127" y="99.06" smashed="yes">
@@
 <attribute name="VALUE" x="86.36" y="-189.23" size="1.778" layer="96"/>
 </instance>
+<instance part="R3" gate="G$1" x="35.56" y="-63.5" smashed="yes" rot="R90">
+<attribute name="R4" x="35.56" y="-63.5" size="1.778" layer="96" rot="R90"/>
+</instance>
+<instance part="LED21" gate="G$1" x="43.18" y="-81.28" smashed="yes">
+<attribute name="VALUE" x="55.88" y="-74.93" size="1.778" layer="96"/>
+</instance>
+<instance part="LED22" gate="G$1" x="43.18" y="-93.98" smashed="yes">
+<attribute name="VALUE" x="55.88" y="-87.63" size="1.778" layer="96"/>
+</instance>
+<instance part="LED23" gate="G$1" x="43.18" y="-106.68" smashed="yes">
+<attribute name="VALUE" x="55.88" y="-100.33" size="1.778" layer="96"/>
+</instance>
+<instance part="LED24" gate="G$1" x="43.18" y="-119.38" smashed="yes">
+<attribute name="VALUE" x="55.88" y="-113.03" size="1.778" layer="96"/>
+</instance>
+<instance part="LED25" gate="G$1" x="43.18" y="-132.08" smashed="yes">
+<attribute name="VALUE" x="55.88" y="-125.73" size="1.778" layer="96"/>
+</instance>
+<instance part="LED26" gate="G$1" x="43.18" y="-144.78" smashed="yes">
+<attribute name="VALUE" x="55.88" y="-138.43" size="1.778" layer="96"/>
+</instance>
+<instance part="LED27" gate="G$1" x="43.18" y="-157.48" smashed="yes">
+<attribute name="VALUE" x="55.88" y="-151.13" size="1.778" layer="96"/>
+</instance>
+<instance part="LED28" gate="G$1" x="43.18" y="-170.18" smashed="yes">
+<attribute name="VALUE" x="55.88" y="-163.83" size="1.778" layer="96"/>
+</instance>
+<instance part="LED29" gate="G$1" x="43.18" y="-182.88" smashed="yes">
+<attribute name="VALUE" x="55.88" y="-176.53" size="1.778" layer="96"/>
+</instance>
+<instance part="LED30" gate="G$1" x="43.18" y="-195.58" smashed="yes">
+<attribute name="VALUE" x="55.88" y="-189.23" size="1.778" layer="96"/>
+</instance>
 </instances>
 <busses>
@@
 <wire x1="66.04" y1="-68.58" x2="66.04" y2="-195.58" width="0.762" layer="92"/>
 <label x="45.72" y="-68.58" size="1.778" layer="95"/>
+</segment>
+<segment>
+<wire x1="35.56" y1="-68.58" x2="35.56" y2="-195.58" width="0.762" layer="92"/>
 </segment>
 </bus>
@@
 <wire x1="121.92" y1="-58.42" x2="121.92" y2="-53.34" width="0.1524" layer="91"/>
 <junction x="121.92" y="-53.34"/>
+<pinref part="R3" gate="G$1" pin="2"/>
 </segment>
 <segment>
@@
 <wire x1="73.66" y1="-195.58" x2="66.04" y2="-195.58" width="0.1524" layer="91"/>
 </segment>
-</net>
+<segment>
+<pinref part="LED21" gate="G$1" pin="K"/>
+<wire x1="43.18" y1="-81.28" x2="35.56" y2="-81.28" width="0.1524" layer="91"/>
+</segment>
+<segment>
+<pinref part="LED22" gate="G$1" pin="K"/>
+<wire x1="43.18" y1="-93.98" x2="35.56" y2="-93.98" width="0.1524" layer="91"/>
+</segment>
+<segment>
+<pinref part="LED23" gate="G$1" pin="K"/>
+<wire x1="43.18" y1="-106.68" x2="35.56" y2="-106.68" width="0.1524" layer="91"/>
+</segment>
+<segment>
+<pinref part="LED24" gate="G$1" pin="K"/>
+<wire x1="43.18" y1="-119.38" x2="35.56" y2="-119.38" width="0.1524" layer="91"/>
+</segment>
+<segment>
+<pinref part="LED25" gate="G$1" pin="K"/>
+<wire x1="43.18" y1="-132.08" x2="35.56" y2="-132.08" width="0.1524" layer="91"/>
+</segment>
+<segment>
+<pinref part="LED26" gate="G$1" pin="K"/>
+<wire x1="43.18" y1="-144.78" x2="35.56" y2="-144.78" width="0.1524" layer="91"/>
+</segment>
+<segment>
+<pinref part="LED27" gate="G$1" pin="K"/>
+<wire x1="43.18" y1="-157.48" x2="35.56" y2="-157.48" width="0.1524" layer="91"/>
+</segment>
+<segment>
+<pinref part="LED29" gate="G$1" pin="K"/>
+<wire x1="43.18" y1="-182.88" x2="35.56" y2="-182.88" width="0.1524" layer="91"/>
+</segment>
+<segment>
+<pinref part="LED28" gate="G$1" pin="K"/>
+<wire x1="43.18" y1="-170.18" x2="35.56" y2="-170.18" width="0.1524" layer="91"/>
+</segment>
+<segment>
+<pinref part="LED30" gate="G$1" pin="K"/>
+<wire x1="43.18" y1="-195.58" x2="35.56" y2="-195.58" width="0.1524" layer="91"/>
+</segment>
+</net>

Commit message: Finish LED
Connections:
- new net N$3: IC6A.Q0, LED21.A
- new net N$30: IC6A.Q1, LED22.A
- new net N$31: IC6A.Q2, LED23.A
- new net N$32: IC6A.Q3, LED24.A
- new net N$33: IC6A.Q4, LED25.A
- new net N$34: IC6A.Q5, LED26.A
- new net N$35: IC6A.Q6, LED27.A
- new net N$36: IC6A.Q7, LED28.A
- new net N$37: IC6A.Q8, LED29.A
- new net N$38: IC6A.Q9, LED30.A
- net 6V: now also R6.2
- net N$1: now also R1.2, R2.2, R5.2, R7.1
- net N$6: now also R6.1, R7.2
- net N$7: now also R4.1
- net N$9: now also R4.2, R5.1
Other:
- moved on the sheet: IC4P, IC6, IC6P

Commit message: modified:   NBPD EAGLE/Layout.s#1 	modified:   NBPD EAGLE/Layout.s#2 	modified:   NBPD EAGLE/Layout.s#3 	modified:   NBPD EAGLE/Layout.s#4 	modified:   NBPD EAGLE/Layout.s#5 	modified:   NBPD EAGLE/Layout.s#6 	modified:   NBPD EAGLE/Layout.s#8 	modified:   NBPD EAGLE/Layout.s#9 	modified:   NBPD EAGLE/Layout.sch
Parts:
- added C1, C10, C2, C3, C4, C5, C6: (no value), resistor:C-US225-062X268
Changed lines of the file:
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@@
 <?xml version="1.0" encoding="utf-8"?>
 <!DOCTYPE eagle SYSTEM "eagle.dtd">
-<eagle version="9.3.0">
+<eagle version="8.4.3">
 <drawing>
 <settings>
@@
 <part name="R4" library="rcl" library_urn="urn:adsk.eagle:library:334" deviceset="R-US_" device="0309/12" package3d_urn="urn:adsk.eagle:package:23571/1" value="220"/>
 <part name="R5" library="rcl" library_urn="urn:adsk.eagle:library:334" deviceset="R-US_" device="0309/12" package3d_urn="urn:adsk.eagle:package:23571/1"/>
-<part name="C1" library="docu-dummy" library_urn="urn:adsk.eagle:library:215" deviceset="C" device=""/>
-<part name="C2" library="docu-dummy" library_urn="urn:adsk.eagle:library:215" deviceset="C" device=""/>
+<part name="C1" library="resistor" library_urn="urn:adsk.eagle:library:348" deviceset="C-US" device="225-062X268" package3d_urn="urn:adsk.eagle:package:26179/1"/>
+<part name="C2" library="resistor" library_urn="urn:adsk.eagle:library:348" deviceset="C-US" device="225-062X268" package3d_urn="urn:adsk.eagle:package:26179/1"/>
 <part name="R6" library="rcl" library_urn="urn:adsk.eagle:library:334" deviceset="R-US_" device="0309/12" package3d_urn="urn:adsk.eagle:package:23571/1"/>
 <part name="R7" library="rcl" library_urn="urn:adsk.eagle:library:334" deviceset="R-US_" device="0309/12" package3d_urn="urn:adsk.eagle:package:23571/1"/>
-<part name="C3" library="docu-dummy" library_urn="urn:adsk.eagle:library:215" deviceset="C" device=""/>
-<part name="C4" library="docu-dummy" library_urn="urn:adsk.eagle:library:215" deviceset="C" device=""/>
-<part name="C5" library="docu-dummy" library_urn="urn:adsk.eagle:library:215" deviceset="C" device=""/>
-<part name="C6" library="docu-dummy" library_urn="urn:adsk.eagle:library:215" deviceset="C" device=""/>
-<part name="C10" library="docu-dummy" library_urn="urn:adsk.eagle:library:215" deviceset="C" device=""/>
+<part name="C3" library="resistor" library_urn="urn:adsk.eagle:library:348" deviceset="C-US" device="225-062X268" package3d_urn="urn:adsk.eagle:package:26179/1"/>
+<part name="C4" library="resistor" library_urn="urn:adsk.eagle:library:348" deviceset="C-US" device="225-062X268" package3d_urn="urn:adsk.eagle:package:26179/1"/>
+<part name="C5" library="resistor" library_urn="urn:adsk.eagle:library:348" deviceset="C-US" device="225-062X268" package3d_urn="urn:adsk.eagle:package:26179/1"/>
+<part name="C6" library="resistor" library_urn="urn:adsk.eagle:library:348" deviceset="C-US" device="225-062X268" package3d_urn="urn:adsk.eagle:package:26179/1"/>
+<part name="C10" library="resistor" library_urn="urn:adsk.eagle:library:348" deviceset="C-US" device="225-062X268" package3d_urn="urn:adsk.eagle:package:26179/1"/>
 <part name="LED1" library="SSL-LX5093TC" deviceset="SSL-LX5093TC" device=""/>
 <part name="LED2" library="SSL-LX5093TC" deviceset="SSL-LX5093TC" device=""/>

Commit message: modified:   NBPD EAGLE/Layout.sch
Parts:
- C1, C10, C2, C3, C4, C5, C6: device resistor:C-US225-062X268 -> rcl:C-US075-063X106
Changed lines of the file:
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@@
 <part name="R4" library="rcl" library_urn="urn:adsk.eagle:library:334" deviceset="R-US_" device="0309/12" package3d_urn="urn:adsk.eagle:package:23571/1" value="220"/>
 <part name="R5" library="rcl" library_urn="urn:adsk.eagle:library:334" deviceset="R-US_" device="0309/12" package3d_urn="urn:adsk.eagle:package:23571/1"/>
-<part name="C1" library="resistor" library_urn="urn:adsk.eagle:library:348" deviceset="C-US" device="225-062X268" package3d_urn="urn:adsk.eagle:package:26179/1"/>
-<part name="C2" library="resistor" library_urn="urn:adsk.eagle:library:348" deviceset="C-US" device="225-062X268" package3d_urn="urn:adsk.eagle:package:26179/1"/>
+<part name="C1" library="rcl" library_urn="urn:adsk.eagle:library:334" deviceset="C-US" device="075-063X106" package3d_urn="urn:adsk.eagle:package:23678/1"/>
+<part name="C2" library="rcl" library_urn="urn:adsk.eagle:library:334" deviceset="C-US" device="075-063X106" package3d_urn="urn:adsk.eagle:package:23678/1"/>
 <part name="R6" library="rcl" library_urn="urn:adsk.eagle:library:334" deviceset="R-US_" device="0309/12" package3d_urn="urn:adsk.eagle:package:23571/1"/>
 <part name="R7" library="rcl" library_urn="urn:adsk.eagle:library:334" deviceset="R-US_" device="0309/12" package3d_urn="urn:adsk.eagle:package:23571/1"/>
-<part name="C3" library="resistor" library_urn="urn:adsk.eagle:library:348" deviceset="C-US" device="225-062X268" package3d_urn="urn:adsk.eagle:package:26179/1"/>
-<part name="C4" library="resistor" library_urn="urn:adsk.eagle:library:348" deviceset="C-US" device="225-062X268" package3d_urn="urn:adsk.eagle:package:26179/1"/>
-<part name="C5" library="resistor" library_urn="urn:adsk.eagle:library:348" deviceset="C-US" device="225-062X268" package3d_urn="urn:adsk.eagle:package:26179/1"/>
-<part name="C6" library="resistor" library_urn="urn:adsk.eagle:library:348" deviceset="C-US" device="225-062X268" package3d_urn="urn:adsk.eagle:package:26179/1"/>
-<part name="C10" library="resistor" library_urn="urn:adsk.eagle:library:348" deviceset="C-US" device="225-062X268" package3d_urn="urn:adsk.eagle:package:26179/1"/>
+<part name="C3" library="rcl" library_urn="urn:adsk.eagle:library:334" deviceset="C-US" device="075-063X106" package3d_urn="urn:adsk.eagle:package:23678/1"/>
+<part name="C4" library="rcl" library_urn="urn:adsk.eagle:library:334" deviceset="C-US" device="075-063X106" package3d_urn="urn:adsk.eagle:package:23678/1"/>
+<part name="C5" library="rcl" library_urn="urn:adsk.eagle:library:334" deviceset="C-US" device="075-063X106" package3d_urn="urn:adsk.eagle:package:23678/1"/>
+<part name="C6" library="rcl" library_urn="urn:adsk.eagle:library:334" deviceset="C-US" device="075-063X106" package3d_urn="urn:adsk.eagle:package:23678/1"/>
+<part name="C10" library="rcl" library_urn="urn:adsk.eagle:library:334" deviceset="C-US" device="075-063X106" package3d_urn="urn:adsk.eagle:package:23678/1"/>
 <part name="LED1" library="SSL-LX5093TC" deviceset="SSL-LX5093TC" device=""/>
 <part name="LED2" library="SSL-LX5093TC" deviceset="SSL-LX5093TC" device=""/>

Commit message: PCB V1
Connections:
- net 10HZGROUND: now also R2.1, R3.1
- net 1HZGROUND: now also R1.1
- net 5V: now also C10.1, C4.1
- net 6V: now also C2.1, C5.1, C6.1
- net N$1: now also C1.2, C10.2, C2.2, C3.2, C4.2, C5.2, C6.2
- net N$7: now also C1.1
- net N$8: now also C3.1

Commit message: PCB V4
Parts:
- added C7, C8, C9: .1uF, rcl:C-US075-063X106
- C1, C4: value (none) -> 1uF
- C10, C3, C5, C6: value (none) -> .1uF
- C2: value (none) -> .33uF
- R5: value (none) -> 330
- R6, R7: value (none) -> 1k
Connections:
- net N$10 renamed LED1
- net N$11 renamed LED2
- net N$12 renamed LED3
- net N$13 renamed LED4
- net N$14 renamed LED5
- net N$15 renamed LED6
- net N$16 renamed LED7
- net N$17 renamed LED8
- net N$18 renamed LED9
- net N$19 renamed LED10
- net N$2 renamed C1K
- net N$20 renamed LED11
- net N$21 renamed LED12
- net N$22 renamed LED13
- net N$23 renamed LED14
- net N$24 renamed LED15
- net N$25 renamed LED16
- net N$26 renamed LED17
- net N$27 renamed LED18
- net N$28 renamed LED19
- net N$29 renamed LED20
- net N$3 renamed LED21
- net N$30 renamed LED22
- net N$31 renamed LED23
- net N$32 renamed LED24
- net N$33 renamed LED25
- net N$34 renamed LED26
- net N$35 renamed LED27
- net N$36 renamed LED28
- net N$37 renamed LED29
- net N$38 renamed LED30
- net N$39 renamed C100
- net N$4 renamed C10
- net N$5 renamed C1
- net N$6 renamed C32
- net N$7 renamed 3.3
- net N$8 renamed 9V
- net N$9 renamed ADJ
- new net 100HZGROUND: LED21.K, LED22.K, LED23.K, LED24.K, LED25.K, LED26.K, LED27.K, LED28.K, LED29.K, LED30.K, R3.1
- new net C512: IC1A.Q6, IC2A.P1
- net 10HZGROUND: no longer LED21.K, LED22.K, LED23.K, LED24.K, LED25.K, LED26.K, LED27.K, LED28.K, LED29.K, LED30.K, R3.1
- net 5V: now also C7.1, C8.1, C9.1, IC5P.VDD
- net N$1: now also C7.2, C8.2, C9.2; no longer IC1A.Q6, IC2A.P1
