File: NBPD EAGLE/Layout.brd (EAGLE design)
At the start: 24.1 x 361.9 mm, 53 parts, among them IC1 4040N, IC2 4040N, IC3 4017N, IC4 4017N, IC5 4017N, IC6 4017N, IC7 7818TV, U1 LM317K, Y1 ACHL-32.768MHZ-EK

Commit message: PCB V1
Parts:
- moved U1 272.3 mm to (135.9, 240.0), flipped to the bottom
- moved IC6 203.4 mm to (133.3, 149.9), flipped to the bottom, turned to 270 degrees
- moved IC4 192.6 mm to (74.9, 171.4), flipped to the bottom, turned to 270 degrees
- moved R5 167.9 mm to (76.2, 106.7), flipped to the bottom
- moved R4 166.4 mm to (86.4, 133.3), flipped to the bottom
- moved R7 161.8 mm to (125.7, 91.4), flipped to the bottom
- moved R6 157.9 mm to (128.3, 50.8), flipped to the bottom
- moved C1 151.8 mm to (33.0, 158.8), flipped to the bottom
- moved C2 136.8 mm to (15.2, 143.5), flipped to the bottom
- moved IC3 127.6 mm to (78.7, 22.9), flipped to the bottom
- moved C10 116.6 mm to (49.5, 87.6), flipped to the bottom
- moved IC1 115.9 mm to (30.5, 25.4), flipped to the bottom
- moved IC5 113.1 mm to (85.1, 85.1), flipped to the bottom, turned to 270 degrees
- moved Y1 103.4 mm to (29.2, 53.3), flipped to the bottom
- moved C3 100.4 mm to (34.3, 149.9), flipped to the bottom
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Routing:
- net N$1: track 0.00 -> 648.7 mm
- net 10HZGROUND: track 0.00 -> 526.0 mm
- net 6V: track 0.00 -> 393.2 mm, vias 0 -> 1
- net 5V: track 0.00 -> 341.5 mm, vias 0 -> 1
- net N$7: track 0.00 -> 302.7 mm, vias 0 -> 1
- net 1HZGROUND: track 0.00 -> 255.6 mm
- net N$6: track 0.00 -> 199.0 mm
- net N$10: track 0.00 -> 181.4 mm
- net N$29: track 0.00 -> 160.6 mm
- net N$9: track 0.00 -> 158.9 mm
- net N$11: track 0.00 -> 152.2 mm
- net N$39: track 0.00 -> 148.6 mm
- net N$38: track 0.00 -> 133.5 mm
- net N$12: track 0.00 -> 131.8 mm
- net N$28: track 0.00 -> 126.5 mm
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Other:
- board size 24.1 x 361.9 mm -> 215.9 x 279.4 mm

Commit message: PCB V2
Parts:
- moved R6 143.5 mm to (27.0, 152.4)
- moved IC2 119.3 mm to (134.9, 46.5), turned to 270 degrees
- moved R7 109.9 mm to (27.0, 139.7)
- moved C10 105.3 mm to (27.0, 190.5)
- moved C2 98.5 mm to (27.0, 241.3)
- moved C1 95.4 mm to (27.0, 254.0)
- moved IC3 89.8 mm to (134.9, 93.0), turned to 270 degrees
- moved C3 79.1 mm to (27.0, 228.6)
- moved C4 78.8 mm to (27.0, 215.9)
- moved C6 78.8 mm to (27.0, 190.5)
- moved C5 77.5 mm to (27.0, 203.2)
- moved R5 76.4 mm to (27.0, 165.1)
- moved R4 74.2 mm to (27.0, 177.8)
- moved IC1 54.7 mm to (81.0, 46.5), turned to 270 degrees
- moved IC7 48.3 mm to (27.0, 127.0)
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Routing:
- net N$1: track 648.7 -> 0.00 mm
- net 10HZGROUND: track 526.0 -> 0.00 mm
- net 6V: track 393.2 -> 0.00 mm, vias 1 -> 0
- net 5V: track 341.5 -> 0.00 mm, vias 1 -> 0
- net N$7: track 302.7 -> 0.00 mm, vias 1 -> 0
- net 1HZGROUND: track 255.6 -> 0.00 mm
- net N$6: track 199.0 -> 0.00 mm
- net N$10: track 181.4 -> 0.00 mm
- net N$29: track 160.6 -> 0.00 mm
- net N$9: track 158.9 -> 0.00 mm
- net N$11: track 152.2 -> 0.00 mm
- net N$39: track 148.6 -> 0.00 mm
- net N$38: track 133.5 -> 0.00 mm
- net N$12: track 131.8 -> 0.00 mm
- net N$28: track 126.5 -> 0.00 mm
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
Commit message: Update POS
Parts:
- moved IC4 46.5 mm to (81.0, 139.7)
- moved IC6 46.5 mm to (134.9, 139.7)
- moved U1 0.95 mm to (134.9, 240.0)

Commit message: PCB V2
Parts:
- moved U1 6.35 mm to (134.9, 246.4)
Routing:
- net N$1: track 0.00 -> 845.4 mm, vias 0 -> 1
- net 10HZGROUND: track 0.00 -> 526.1 mm
- net 6V: track 0.00 -> 462.3 mm, vias 0 -> 1
- net 5V: track 0.00 -> 441.7 mm, vias 0 -> 1
- net N$7: track 0.00 -> 302.1 mm
- net 1HZGROUND: track 0.00 -> 244.1 mm
- net N$10: track 0.00 -> 178.0 mm
- net N$6: track 0.00 -> 161.4 mm
- net N$9: track 0.00 -> 154.7 mm, vias 0 -> 1
- net N$11: track 0.00 -> 144.4 mm
- net N$12: track 0.00 -> 123.6 mm
- net N$29: track 0.00 -> 122.7 mm, vias 0 -> 1
- net N$38: track 0.00 -> 122.7 mm
- net N$3: track 0.00 -> 120.9 mm
- net N$20: track 0.00 -> 120.7 mm
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Other:
- board text added: "5V"
- board text added: "6V"
- board text added: "GND"

Commit message: PCB V4
Parts:
- added C7, C8, C9: .1uF, rcl:C075-063X106
- C1, C4: value (none) -> 1uF
- C10, C3, C5, C6: value (none) -> .1uF
- C2: value (none) -> .33uF
- R5: value (none) -> 330
- R6, R7: value (none) -> 1k
- moved R2 71.7 mm to (81.0, 76.2)
- moved R3 69.0 mm to (134.9, 76.2), turned to 0 degrees
- moved R1 64.4 mm to (81.0, 71.1)
- moved R4 50.8 mm to (27.0, 127.0), turned to 180 degrees
- moved R6 50.8 mm to (27.0, 101.6)
- moved IC7 50.8 mm to (27.0, 76.2)
- moved R5 50.8 mm to (27.0, 114.3)
- moved R7 50.8 mm to (27.0, 88.9), turned to 180 degrees
- moved IC5 48.0 mm to (81.0, 141.0)
- moved IC3 46.7 mm to (134.9, 139.7)
- moved IC1 46.5 mm to (81.0, 93.0)
- moved IC2 46.5 mm to (134.9, 93.0)
- moved IC4 46.5 mm to (81.0, 186.2)
- moved IC6 46.5 mm to (134.9, 186.2)
- moved C10 12.7 mm to (27.0, 177.8)
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Connections:
- net N$10 renamed LED1
- net N$11 renamed LED2
- net N$12 renamed LED3
- net N$13 renamed LED4
- net N$14 renamed LED5
- net N$15 renamed LED6
- net N$16 renamed LED7
- net N$17 renamed LED8
- net N$18 renamed LED9
- net N$19 renamed LED10
- net N$2 renamed C1K
- net N$20 renamed LED11
- net N$21 renamed LED12
- net N$22 renamed LED13
- net N$23 renamed LED14
- net N$24 renamed LED15
- net N$25 renamed LED16
- net N$26 renamed LED17
- net N$27 renamed LED18
- net N$28 renamed LED19
- net N$29 renamed LED20
- net N$3 renamed LED21
- net N$30 renamed LED22
- net N$31 renamed LED23
- net N$32 renamed LED24
- net N$33 renamed LED25
- net N$34 renamed LED26
- net N$35 renamed LED27
- net N$36 renamed LED28
- net N$37 renamed LED29
- net N$38 renamed LED30
- net N$39 renamed C100
- net N$4 renamed C10
- net N$5 renamed C1
- net N$6 renamed C32
- net N$7 renamed 3.3
- net N$8 renamed 9V
- net N$9 renamed ADJ
- removed net VDD: IC5.16
- new net 100HZGROUND: LED21.1, LED22.1, LED23.1, LED24.1, LED25.1, LED26.1, LED27.1, LED28.1, LED29.1, LED30.1, R3.1
- new net C512: IC1.2, IC2.10
- net 10HZGROUND: no longer LED21.1, LED22.1, LED23.1, LED24.1, LED25.1, LED26.1, LED27.1, LED28.1, LED29.1, LED30.1, R3.1
- net 5V: now also C7.1, C8.1, C9.1, IC5.16
- net N$1: now also C7.2, C8.2, C9.2; no longer IC1.2, IC2.10
Routing:
- net 10HZGROUND: track 526.1 -> 251.8 mm
- net 100HZGROUND: track 0.00 -> 251.0 mm
- net 9V: track 104.7 -> 324.2 mm, vias 0 -> 3
- net N$1: track 845.4 -> 740.9 mm, vias 1 -> 3
- net 5V: track 441.7 -> 342.6 mm, vias 1 -> 0
- net C32: track 161.4 -> 93.6 mm
- net ADJ: track 154.7 -> 214.9 mm, vias 1 -> 0
- net LED9: track 43.4 -> 103.2 mm
- net LED28: track 68.8 -> 128.2 mm
- net C512: track 0.00 -> 51.6 mm
- net LED5: track 83.3 -> 31.8 mm
- net LED1: track 178.0 -> 128.9 mm
- net LED16: track 30.9 -> 79.5 mm
- net LED10: track 77.1 -> 125.5 mm, vias 0 -> 1
- net LED30: track 122.7 -> 170.6 mm
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Other:
- board text added: "9V"
- board text removed: "5V"

Commit message: trace widen
Parts:
- moved C10 171.7 mm to (188.9, 120.7)
- moved C6 168.8 mm to (188.9, 142.9)
- moved Y1 168.1 mm to (188.9, 98.4)
- moved C5 166.1 mm to (188.9, 165.1)
- moved C4 164.4 mm to (188.9, 187.3)
- moved C3 163.0 mm to (188.9, 209.6)
- moved C2 162.2 mm to (188.9, 231.8)
- moved C1 161.9 mm to (188.9, 254.0)
- moved C7 88.9 mm to (27.0, 254.0)
- moved C8 79.4 mm to (27.0, 231.8)
- moved C9 69.9 mm to (27.0, 209.6)
- moved R4 60.3 mm to (27.0, 187.3)
- moved R5 50.8 mm to (27.0, 165.1)
- moved R6 41.3 mm to (27.0, 142.9)
- moved R7 31.8 mm to (27.0, 120.7)
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Routing:
- net N$1: track 740.9 -> 0.00 mm, vias 3 -> 0
- net 6V: track 480.2 -> 0.00 mm, vias 4 -> 0
- net 5V: track 342.6 -> 0.00 mm
- net 9V: track 324.2 -> 0.00 mm, vias 3 -> 0
- net 3.3: track 309.5 -> 0.00 mm
- net 1HZGROUND: track 282.4 -> 0.00 mm
- net 10HZGROUND: track 251.8 -> 0.00 mm
- net 100HZGROUND: track 251.0 -> 0.00 mm
- net ADJ: track 214.9 -> 0.00 mm
- net LED30: track 170.6 -> 0.00 mm
- net LED20: track 170.1 -> 0.00 mm
- net LED19: track 138.7 -> 0.00 mm
- net LED29: track 138.7 -> 0.00 mm
- net LED1: track 128.9 -> 0.00 mm
- net LED28: track 128.2 -> 0.00 mm
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
Commit message: autoroute
Routing:
- net N$1: track 0.00 -> 817.4 mm
- net 5V: track 0.00 -> 532.7 mm, vias 0 -> 1
- net 6V: track 0.00 -> 401.3 mm
- net 3.3: track 0.00 -> 393.5 mm
- net 9V: track 0.00 -> 266.4 mm, vias 0 -> 1
- net 1HZGROUND: track 0.00 -> 262.8 mm
- net 10HZGROUND: track 0.00 -> 252.5 mm
- net 100HZGROUND: track 0.00 -> 251.8 mm
- net C32: track 0.00 -> 205.7 mm, vias 0 -> 2
- net LED20: track 0.00 -> 182.4 mm, vias 0 -> 1
- net LED30: track 0.00 -> 176.7 mm, vias 0 -> 1
- net ADJ: track 0.00 -> 172.4 mm
- net LED1: track 0.00 -> 147.8 mm, vias 0 -> 1
- net LED19: track 0.00 -> 143.6 mm, vias 0 -> 1
- net LED29: track 0.00 -> 138.8 mm, vias 0 -> 1
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