File: NBPD EAGLE/Layout.brd (EAGLE design)
At the start: 215.9 x 279.4 mm, 56 parts, among them IC1 4040N, IC2 4040N, IC3 4017N, IC4 4017N, IC5 4017N, IC6 4017N, IC7 7818TV, U1 LM317K, Y1 ACHL-32.768MHZ-EK

Commit message: final
Routing:
- net 9V: track 266.4 -> 525.0 mm, vias 1 -> 4
- net 6V: track 401.3 -> 493.5 mm, vias 0 -> 3
- net N$1: track 817.4 -> 873.3 mm, vias 0 -> 3
Changed lines of the file:
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@@
 <wire x1="185.42" y1="231.775" x2="185.1025" y2="231.775" width="1.524" layer="1"/>
 <wire x1="185.42" y1="210.185" x2="185.1025" y2="209.55" width="1.524" layer="1"/>
-<wire x1="185.42" y1="232.41" x2="185.42" y2="254" width="1.524" layer="1"/>
-<wire x1="185.42" y1="254" x2="185.1025" y2="254" width="1.524" layer="1"/>
-<wire x1="185.42" y1="232.41" x2="185.1025" y2="231.775" width="1.524" layer="1"/>
 <wire x1="148.59" y1="120.65" x2="139.065" y2="130.175" width="1.524" layer="16"/>
 <wire x1="185.1025" y1="120.65" x2="148.59" y2="120.65" width="1.524" layer="16"/>
@@
 <wire x1="138.43" y1="130.81" x2="138.7475" y2="130.81" width="1.524" layer="1"/>
 <wire x1="131.445" y1="88.9" x2="131.1275" y2="89.154" width="1.524" layer="1"/>
+<via x="189.23" y="265.43" extent="1-16" drill="0.65" shape="square"/>
+<via x="191.77" y="265.43" extent="1-16" drill="0.65" shape="square"/>
+<via x="194.31" y="265.43" extent="1-16" drill="0.65" shape="square"/>
+<wire x1="194.31" y1="265.43" x2="194.31" y2="255.64539375" width="1.524" layer="16"/>
+<wire x1="194.31" y1="255.64539375" x2="195.0085" y2="254.94689375" width="1.524" layer="16"/>
+<wire x1="195.0085" y1="254.94689375" x2="195.0085" y2="219.456" width="1.524" layer="16"/>
+<wire x1="195.0085" y1="219.456" x2="185.1025" y2="209.55" width="1.524" layer="16"/>
+<wire x1="194.31" y1="265.43" x2="191.77" y2="265.43" width="1.524" layer="16"/>
+<wire x1="191.77" y1="265.43" x2="189.23" y2="265.43" width="1.524" layer="16"/>
+<wire x1="189.23" y1="265.43" x2="189.23" y2="258.1275" width="1.524" layer="16"/>
+<wire x1="189.23" y1="258.1275" x2="185.1025" y2="254" width="1.524" layer="16"/>
 </signal>
 <signal name="C1K">
@@
 <wire x1="192.7225" y1="142.875" x2="189.865" y2="142.875" width="1.524" layer="16"/>
 <wire x1="131.445" y1="102.235" x2="131.1275" y2="101.854" width="1.524" layer="16"/>
+<via x="181.61" y="265.43" extent="1-16" drill="0.65" shape="square"/>
+<via x="184.15" y="265.43" extent="1-16" drill="0.65" shape="square"/>
+<via x="186.69" y="265.43" extent="1-16" drill="0.65" shape="square"/>
+<wire x1="181.61" y1="265.43" x2="172.466" y2="256.286" width="1.524" layer="1"/>
+<wire x1="149.80210625" y1="246.38" x2="138.6459" y2="246.38" width="1.524" layer="1"/>
+<wire x1="172.466" y1="256.286" x2="159.70810625" y2="256.286" width="1.524" layer="1"/>
+<wire x1="159.70810625" y1="256.286" x2="149.80210625" y2="246.38" width="1.524" layer="1"/>
+<wire x1="186.69" y1="237.49" x2="192.405" y2="231.775" width="1.524" layer="1"/>
+<wire x1="186.69" y1="265.43" x2="186.69" y2="255.07065625" width="1.524" layer="1"/>
+<wire x1="186.69" y1="255.07065625" x2="186.9821" y2="254.77855625" width="1.524" layer="1"/>
+<wire x1="186.9821" y1="254.77855625" x2="186.9821" y2="253.22144375" width="1.524" layer="1"/>
+<wire x1="186.9821" y1="253.22144375" x2="186.69" y2="252.92934375" width="1.524" layer="1"/>
+<wire x1="186.69" y1="252.92934375" x2="186.69" y2="237.49" width="1.524" layer="1"/>
+<wire x1="181.61" y1="265.43" x2="184.15" y2="265.43" width="1.524" layer="1"/>
+<wire x1="184.15" y1="265.43" x2="186.69" y2="265.43" width="1.524" layer="1"/>
 </signal>
 <signal name="3.3">
@@
 <wire x1="29.845" y1="95.885" x2="29.5275" y2="95.885" width="1.524" layer="1"/>
 <via x="48.26" y="208.28" extent="1-16" drill="0.35"/>
+<via x="173.99" y="265.43" extent="1-16" drill="0.65" shape="square"/>
+<via x="176.53" y="265.43" extent="1-16" drill="0.65" shape="square"/>
+<via x="179.07" y="265.43" extent="1-16" drill="0.65" shape="square"/>
+<wire x1="179.07" y1="265.43" x2="176.53" y2="265.43" width="1.524" layer="1"/>
+<wire x1="176.53" y1="265.43" x2="173.99" y2="265.43" width="1.524" layer="1"/>
+<wire x1="173.99" y1="265.43" x2="105.41" y2="265.43" width="1.524" layer="1"/>
+<wire x1="51.75810625" y1="256.286" x2="48.514" y2="253.04189375" width="1.524" layer="1"/>
+<wire x1="48.514" y1="208.534" x2="48.26" y2="208.28" width="1.524" layer="1"/>
+<wire x1="48.514" y1="253.04189375" x2="48.514" y2="208.534" width="1.524" layer="1"/>
+<wire x1="105.41" y1="265.43" x2="96.266" y2="256.286" width="1.524" layer="1"/>
+<wire x1="96.266" y1="256.286" x2="51.75810625" y2="256.286" width="1.524" layer="1"/>
+<wire x1="192.7225" y1="209.55" x2="192.7225" y2="213.93710625" width="1.524" layer="16"/>
+<wire x1="192.7225" y1="213.93710625" x2="197.2945" y2="218.50910625" width="1.524" layer="16"/>
+<wire x1="197.2945" y1="218.50910625" x2="197.2945" y2="265.67839375" width="1.524" layer="16"/>
+<wire x1="197.2945" y1="265.67839375" x2="195.25689375" y2="267.716" width="1.524" layer="16"/>
+<wire x1="195.25689375" y1="267.716" x2="181.54644375" y2="267.716" width="1.524" layer="16"/>
+<wire x1="179.26044375" y1="265.43" x2="179.07" y2="265.43" width="1.524" layer="16"/>
+<wire x1="181.54644375" y1="267.716" x2="179.26044375" y2="265.43" width="1.524" layer="16"/>
 </signal>
 <signal name="ADJ">
@@
 <wire x1="130.81" y1="86.36" x2="131.1275" y2="86.614" width="1.524" layer="16"/>
 </signal>
-<signal name="N$4">
-<via x="191.77" y="265.43" extent="1-16" drill="0.65" shape="square"/>
-<via x="194.31" y="265.43" extent="1-16" drill="0.65" shape="square"/>
-</signal>
-<signal name="N$5">
-<via x="189.23" y="265.43" extent="1-16" drill="0.65" shape="square"/>
-</signal>
-<signal name="N$6">
-<via x="186.69" y="265.43" extent="1-16" drill="0.65" shape="square"/>
-</signal>
-<signal name="N$7">
-<via x="184.15" y="265.43" extent="1-16" drill="0.65" shape="square"/>
-</signal>
-<signal name="N$8">
-<via x="181.61" y="265.43" extent="1-16" drill="0.65" shape="square"/>
-</signal>
-<signal name="N$9">
-<via x="179.07" y="265.43" extent="1-16" drill="0.65" shape="square"/>
-</signal>
-<signal name="N$10">
-<via x="173.99" y="265.43" extent="1-16" drill="0.65" shape="square"/>
-</signal>
-<signal name="N$2">
-<via x="176.53" y="265.43" extent="1-16" drill="0.65" shape="square"/>
-</signal>
 </signals>

Commit message: rev3 final
Routing:
- net 9V: track 525.0 -> 344.8 mm
- net 6V: track 493.5 -> 415.1 mm, vias 3 -> 5
- net LED3: track 90.4 -> 105.7 mm, vias 0 -> 2
- net LED2: track 118.3 -> 133.6 mm, vias 1 -> 4
- net LED17: track 96.9 -> 112.1 mm, vias 1 -> 2
- net 5V: track 532.7 -> 518.7 mm, vias 1 -> 3
- net 3.3: track 393.5 -> 380.8 mm
- net LED25: track 61.8 -> 51.4 mm
- net LED7: track 88.4 -> 79.5 mm, vias 0 -> 1
- net LED8: track 95.4 -> 87.3 mm, vias 1 -> 2
- net LED28: track 135.2 -> 142.5 mm
- net LED16: track 88.7 -> 82.2 mm, vias 0 -> 1
- net LED1: track 147.8 -> 153.2 mm, vias 1 -> 5
- net LED19: track 143.6 -> 148.8 mm, vias 1 -> 2
- net LED15: track 45.3 -> 50.4 mm
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
Commit message: Schematic Labels & PDF Names
Parts:
- C3: value .1uF -> 0.33uF
Changed lines of the file:
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@@
 <attribute name="VALUE" x="199.7075" y="231.775" size="1.27" layer="28" ratio="10" rot="MR0"/>
 </element>
-<element name="C3" library="rcl" library_urn="urn:adsk.eagle:library:334" package="C075-063X106" package3d_urn="urn:adsk.eagle:package:23678/1" value=".1uF" x="188.9125" y="209.55" smashed="yes" rot="MR0">
+<element name="C3" library="rcl" library_urn="urn:adsk.eagle:library:334" package="C075-063X106" package3d_urn="urn:adsk.eagle:package:23678/1" value="0.33uF" x="188.9125" y="209.55" smashed="yes" rot="MR0">
 <attribute name="NAME" x="197.5485" y="211.709" size="1.27" layer="26" ratio="10" rot="MR0"/>
 <attribute name="VALUE" x="198.4375" y="209.55" size="1.27" layer="28" ratio="10" rot="MR0"/>
@@
 </element>
 <element name="C5" library="rcl" library_urn="urn:adsk.eagle:library:334" package="C075-063X106" package3d_urn="urn:adsk.eagle:package:23678/1" value=".1uF" x="188.9125" y="165.1" smashed="yes" rot="MR0">
+<attribute name="C5" value="0.1uF" x="188.9125" y="165.1" size="1.778" layer="28" rot="MR0" display="off"/>
 <attribute name="NAME" x="198.8185" y="167.259" size="1.27" layer="26" ratio="10" rot="MR0"/>
+<attribute name="SPICEPREFIX" value="C" x="188.9125" y="165.1" size="1.778" layer="28" rot="MR0" display="off"/>
 <attribute name="VALUE" x="198.4375" y="165.1" size="1.27" layer="28" ratio="10" rot="MR0"/>
 </element>
@@
 <element name="IC7" library="linear" library_urn="urn:adsk.eagle:library:262" package="TO220V" package3d_urn="urn:adsk.eagle:package:16417/1" value="7818TV" x="26.9875" y="98.425" smashed="yes" rot="MR0">
 <attribute name="NAME" x="23.1775" y="91.1098" size="1.27" layer="26" ratio="10" rot="MR0"/>
+<attribute name="SPICEPREFIX" value="J" x="26.9875" y="98.425" size="1.778" layer="28" rot="MR0" display="off"/>
 <attribute name="VALUE" x="32.0675" y="90.805" size="1.27" layer="28" ratio="10" rot="MR0"/>
 </element>
@@
 <element name="R1" library="rcl" library_urn="urn:adsk.eagle:library:334" package="0207/12" package3d_urn="urn:adsk.eagle:package:23489/1" value="220" x="80.9625" y="71.12" smashed="yes" rot="MR0">
 <attribute name="NAME" x="77.7875" y="67.8942" size="1.27" layer="26" ratio="10" rot="MR0"/>
-<attribute name="R6" value="220" x="30.1625" y="-33.02" size="1.778" layer="28" rot="MR0" display="off"/>
 <attribute name="VALUE" x="85.7885" y="67.8942" size="1.27" layer="28" ratio="10" rot="MR0"/>
 </element>
 <element name="R2" library="rcl" library_urn="urn:adsk.eagle:library:334" package="0207/12" package3d_urn="urn:adsk.eagle:package:23489/1" value="220" x="80.9625" y="76.2" smashed="yes" rot="MR0">
 <attribute name="NAME" x="77.7875" y="78.867" size="1.27" layer="26" ratio="10" rot="MR0"/>
-<attribute name="R5" value="220" x="14.9225" y="-27.94" size="1.778" layer="28" rot="MR0" display="off"/>
 <attribute name="VALUE" x="84.5185" y="78.867" size="1.27" layer="28" ratio="10" rot="MR0"/>
 </element>
 <element name="R3" library="rcl" library_urn="urn:adsk.eagle:library:334" package="0207/12" package3d_urn="urn:adsk.eagle:package:23489/1" value="220" x="134.9375" y="76.2" smashed="yes" rot="MR0">
 <attribute name="NAME" x="133.0325" y="72.517" size="1.27" layer="26" ratio="10" rot="MR0"/>
-<attribute name="R4" value="220" x="53.6575" y="-27.94" size="1.778" layer="28" rot="MR0" display="off"/>
 <attribute name="VALUE" x="138.4935" y="72.517" size="1.27" layer="28" ratio="10" rot="MR0"/>
 </element>

Commit message: 3.3V Update
Parts:
- removed R4: 220, rcl:0309/12
- removed R5: 330, rcl:0309/12
- removed U1: LM317K, LM317K:TO1090P3010X870-4P
- added IC8: 786TV, linear:TO220V
Connections:
- removed net ADJ: R4.2, R5.1, U1.1
- net 3.3: now also IC8.3; no longer R4.1, U1.3
- net 6V: now also IC8.1; no longer U1.2
- net N$1: now also IC8.2; no longer R5.2
Routing:
- net ADJ: track 171.3 -> 0.00 mm
- net 3.3: track 380.8 -> 257.4 mm
- net N$1: track 877.0 -> 994.8 mm
- net 6V: track 415.1 -> 428.8 mm
Changed lines of the file:
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@@
 <attribute name="VALUE" x="138.4935" y="72.517" size="1.27" layer="28" ratio="10" rot="MR0"/>
-</element>
-<element name="R4" library="rcl" library_urn="urn:adsk.eagle:library:334" package="0309/12" package3d_urn="urn:adsk.eagle:package:23571/1" value="220" x="26.9875" y="187.325" smashed="yes" rot="MR180">
-<attribute name="NAME" x="24.0665" y="184.15" size="1.27" layer="26" ratio="10" rot="MR180"/>
-<attribute name="SPICEPREFIX" value="R" x="26.9875" y="187.325" size="1.778" layer="28" rot="MR180" display="off"/>
-<attribute name="VALUE" x="28.8925" y="184.2008" size="1.27" layer="28" ratio="10" rot="MR180"/>
-</element>
-<element name="R5" library="rcl" library_urn="urn:adsk.eagle:library:334" package="0309/12" package3d_urn="urn:adsk.eagle:package:23571/1" value="330" x="26.9875" y="165.1" smashed="yes" rot="MR0">
-<attribute name="NAME" x="24.8285" y="160.655" size="1.27" layer="26" ratio="10" rot="MR0"/>
-<attribute name="SPICEPREFIX" value="R" x="26.9875" y="165.1" size="1.778" layer="28" rot="MR0" display="off"/>
-<attribute name="VALUE" x="30.1625" y="160.6042" size="1.27" layer="28" ratio="10" rot="MR0"/>
 </element>
 <element name="R6" library="rcl" library_urn="urn:adsk.eagle:library:334" package="0309/12" package3d_urn="urn:adsk.eagle:package:23571/1" value="1k" x="26.9875" y="142.875" smashed="yes" rot="MR0">
@@
 <attribute name="SPICEPREFIX" value="R" x="26.9875" y="120.65" size="1.778" layer="28" rot="MR180" display="off"/>
 <attribute name="VALUE" x="28.8925" y="117.5258" size="1.27" layer="28" ratio="10" rot="MR180"/>
-</element>
-<element name="U1" library="LM317K" package="TO1090P3010X870-4P" value="LM317K" x="134.9375" y="246.38" smashed="yes" rot="MR0">
-<attribute name="DESCRIPTION" value="Voltage regulators" x="103.1875" y="220.98" size="1.778" layer="28" rot="MR0" display="off"/>
-<attribute name="HEIGHT" value="mm" x="134.9375" y="246.38" size="1.778" layer="28" rot="MR0" display="off"/>
-<attribute name="MANUFACTURER_NAME" value="STMicroelectronics" x="134.9375" y="246.38" size="1.778" layer="28" rot="MR0" display="off"/>
-<attribute name="MANUFACTURER_PART_NUMBER" value="LM317K" x="134.9375" y="246.38" size="1.778" layer="28" rot="MR0" display="off"/>
-<attribute name="MOUSER_PART_NUMBER" value="511-LM317K" x="134.9375" y="246.38" size="1.778" layer="28" rot="MR0" display="off"/>
-<attribute name="MOUSER_PRICE-STOCK" value="https://www.mouser.com/Search/Refine.aspx?Keyword=511-LM317K" x="134.9375" y="246.38" size="1.778" layer="28" rot="MR0" display="off"/>
-<attribute name="NAME" x="141.449690625" y="256.9369" size="2.085940625" layer="26" ratio="10" rot="SMR0"/>
-<attribute name="RS_PART_NUMBER" value="7140786" x="134.9375" y="246.38" size="1.778" layer="28" rot="MR0" display="off"/>
-<attribute name="RS_PRICE-STOCK" value="https://uk.rs-online.com/web/p/products/7140786" x="134.9375" y="246.38" size="1.778" layer="28" rot="MR0" display="off"/>
-<attribute name="VALUE" x="141.59475" y="222.9272" size="2.08356875" layer="28" ratio="10" rot="SMR0"/>
 </element>
 <element name="Y1" library="ACHL-32.768MHZ-EK" package="ACHL" value="ACHL-32.768MHZ-EK" x="188.9125" y="98.425" smashed="yes" rot="MR0">
@@
 <attribute name="VALUE" x="36.5125" y="209.55" size="1.27" layer="28" ratio="10" rot="MR0"/>
 </element>
+<element name="IC8" library="linear" library_urn="urn:adsk.eagle:library:262" package="TO220V" package3d_urn="urn:adsk.eagle:package:16417/2" value="786TV" x="129.54" y="256.54" smashed="yes">
+<attribute name="NAME" x="124.46" y="250.4948" size="1.27" layer="25" ratio="10"/>
+<attribute name="VALUE" x="124.46" y="248.92" size="1.27" layer="27" ratio="10"/>
+</element>
 </elements>
 <signals>
@@
 <contactref element="R1" pad="2"/>
 <contactref element="R2" pad="2"/>
-<contactref element="R5" pad="2"/>
 <contactref element="R7" pad="1"/>
 <contactref element="R3" pad="2"/>
@@
 <wire x1="26.9875" y1="95.885" x2="26.9875" y2="114.3" width="1.524" layer="1"/>
 <wire x1="23.1775" y1="167.64" x2="22.70125" y2="167.16375" width="1.524" layer="1"/>
-<wire x1="22.70125" y1="167.16375" x2="20.6375" y2="165.1" width="1.524" layer="1"/>
 <wire x1="23.1775" y1="209.55" x2="23.1775" y2="167.64" width="1.524" layer="1"/>
 <wire x1="23.1775" y1="209.55" x2="23.1775" y2="231.775" width="1.524" layer="1"/>
@@
 <wire x1="139.3825" y1="84.1375" x2="174.625" y2="84.1375" width="1.524" layer="16"/>
 <wire x1="139.3825" y1="84.1375" x2="138.7475" y2="84.074" width="1.524" layer="16"/>
+<contactref element="IC8" pad="2"/>
+<wire x1="129.54" y1="254" x2="129.54" y2="264.16" width="1.524" layer="1"/>
+<wire x1="129.54" y1="264.16" x2="33.3375" y2="264.16" width="1.524" layer="1"/>
+<wire x1="33.3375" y1="264.16" x2="23.1775" y2="254" width="1.524" layer="1"/>
 </signal>
 <signal name="C1K">
@@
 </signal>
 <signal name="6V">
-<contactref element="U1" pad="2"/>
 <contactref element="R6" pad="2"/>
 <contactref element="C2" pad="1"/>
@@
 <wire x1="180.81625" y1="264.16" x2="180.81625" y2="264.31875" width="1.524" layer="1"/>
 <wire x1="173.19625" y1="256.54" x2="180.81625" y2="264.16" width="1.524" layer="1"/>
-<wire x1="138.7475" y1="256.54" x2="173.19625" y2="256.54" width="1.524" layer="1"/>
-<wire x1="138.7475" y1="246.38" x2="138.7475" y2="256.54" width="1.524" layer="1"/>
+<wire x1="173.19625" y1="256.54" x2="138.7475" y2="256.54" width="1.524" layer="1"/>
 <wire x1="181.2925" y1="264.795" x2="181.61" y2="265.43" width="1.524" layer="1"/>
-<wire x1="138.7475" y1="246.38" x2="138.6459" y2="246.38" width="1.524" layer="1"/>
 <wire x1="177.95875" y1="246.53875" x2="192.7225" y2="231.775" width="1.524" layer="16"/>
 <wire x1="173.51375" y1="250.98375" x2="177.95875" y2="246.53875" width="1.524" layer="1"/>
@@
 <via x="177.95875" y="246.53875" extent="1-16" drill="0.35"/>
 <via x="132.55625" y="109.06125" extent="1-16" drill="0.35"/>
+<contactref element="IC8" pad="1"/>
+<wire x1="127" y1="247.904" x2="127" y2="254" width="1.524" layer="1"/>
+<wire x1="134.40210625" y1="247.904" x2="127" y2="247.904" width="1.524" layer="1"/>
+<wire x1="138.7475" y1="252.24939375" x2="134.40210625" y2="247.904" width="1.524" layer="1"/>
+<wire x1="138.7475" y1="256.54" x2="138.7475" y2="252.24939375" width="1.524" layer="1"/>
 </signal>
 <signal name="3.3">
 <contactref element="Y1" pad="8"/>
-<contactref element="U1" pad="3"/>
 <contactref element="Y1" pad="1"/>
-<contactref element="R4" pad="1"/>
 <contactref element="C1" pad="1"/>
 <wire x1="192.7225" y1="102.235" x2="192.7225" y2="94.615" width="1.524" layer="1"/>
-<wire x1="25.87625" y1="192.56375" x2="20.6375" y2="187.325" width="1.524" layer="16"/>
-<wire x1="25.87625" y1="226.06" x2="25.87625" y2="192.56375" width="1.524" layer="16"/>
-<wire x1="100.48875" y1="226.06" x2="25.87625" y2="226.06" width="1.524" layer="16"/>
-<wire x1="115.2525" y1="240.82375" x2="100.48875" y2="226.06" width="1.524" layer="16"/>
-<wire x1="121.6025" y1="240.82375" x2="115.2525" y2="240.82375" width="1.524" layer="16"/>
-<wire x1="121.6025" y1="240.82375" x2="121.7041" y2="240.919" width="1.524" layer="16"/>
-<wire x1="187.6425" y1="248.92" x2="192.7225" y2="254" width="1.524" layer="16"/>
-<wire x1="129.69875" y1="248.92" x2="187.6425" y2="248.92" width="1.524" layer="16"/>
-<wire x1="122.2375" y1="241.45875" x2="129.69875" y2="248.92" width="1.524" layer="16"/>
-<wire x1="122.2375" y1="241.45875" x2="121.7041" y2="240.919" width="1.524" layer="16"/>
 <wire x1="195.2625" y1="105.0925" x2="193.04" y2="102.87" width="1.524" layer="1"/>
 <wire x1="195.2625" y1="251.46" x2="195.2625" y2="105.0925" width="1.524" layer="1"/>
 <wire x1="192.7225" y1="254" x2="195.2625" y2="251.46" width="1.524" layer="1"/>
 <wire x1="193.04" y1="102.87" x2="192.7225" y2="102.235" width="1.524" layer="1"/>
+<contactref element="IC8" pad="3"/>
+<wire x1="196.99674375" y1="272.43158125" x2="196.10400625" y2="273.32431875" width="1.524" layer="1"/>
+<wire x1="135.26060625" y1="261.366" x2="132.08" y2="258.18539375" width="1.524" layer="1"/>
+<wire x1="132.08" y1="258.18539375" x2="132.08" y2="254" width="1.524" layer="1"/>
+<wire x1="196.99674375" y1="262.66135" x2="196.99674375" y2="272.43158125" width="1.524" layer="1"/>
+<wire x1="156.99775625" y1="261.366" x2="135.26060625" y2="261.366" width="1.524" layer="1"/>
+<wire x1="168.956075" y1="273.32431875" x2="156.99775625" y2="261.366" width="1.524" layer="1"/>
+<wire x1="192.7225" y1="254" x2="192.7225" y2="258.38710625" width="1.524" layer="1"/>
+<wire x1="192.7225" y1="258.38710625" x2="196.99674375" y2="262.66135" width="1.524" layer="1"/>
+<wire x1="196.10400625" y1="273.32431875" x2="168.956075" y2="273.32431875" width="1.524" layer="1"/>
 </signal>
 <signal name="9V">
@@
 <wire x1="192.0875" y1="209.2325" x2="192.7225" y2="209.55" width="1.524" layer="16"/>
 </signal>
-<signal name="ADJ">
-<contactref element="U1" pad="1"/>
-<contactref element="R4" pad="2"/>
-<contactref element="R5" pad="1"/>
-<wire x1="123.34875" y1="220.18625" x2="138.6459" y2="235.4834" width="1.524" layer="16"/>
-<wire x1="37.7825" y1="220.18625" x2="123.34875" y2="220.18625" width="1.524" layer="16"/>
-<wire x1="28.2575" y1="210.66125" x2="37.7825" y2="220.18625" width="1.524" layer="16"/>
-<wire x1="28.2575" y1="187.325" x2="28.2575" y2="210.66125" width="1.524" layer="16"/>
-<wire x1="33.3375" y1="187.325" x2="28.2575" y2="187.325" width="1.524" layer="16"/>
-<wire x1="33.3375" y1="187.325" x2="33.3375" y2="165.1" width="1.524" layer="1"/>
-</signal>
 <signal name="LED1">
